Commit message: refactor moveit config

File: src/lion_robot_description/urdf/robot_w_screwdriver.urdf (robot description, URDF)
Before this commit: robot lion_robot_description, 13 links, 12 joints
Links:
- added link vacuum_tcp
Joints:
- added joint screwdriver-vacuum_tcp: type fixed, parent screwdriver, child vacuum_tcp, origin xyz=0.0 0.0 -0.3 rpy=0 0 0
